File: 12v-switch.brd (EAGLE design)
At the start: 50 x 50 mm, 18 parts, among them J1 En, J2 Bypass, J3 POWERPOLE_POWER25A, J4 12v, J5 12V Out, J6 POWERPOLE_POWER25A, J7 LEN EN, Q1 SI4532ADY

Commit message: output power poles are now compatible with horizontal ones as well as vertical
Parts:
- moved F1 5.08 mm to (36.8, 25.4)
- turned J6 to 90 degrees
Routing:
- net 12V-SWITCHED: track 31.2 -> 17.7 mm
- net N$95: track 32.3 -> 27.2 mm
Changed lines of the file:
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@@
 </autorouter>
 <elements>
-<element name="LED2" library="led" package="CHIP-LED0805" value="En" x="11.43" y="10.16" rot="R180"/>
+<element name="LED2" library="led" package="CHIP-LED0805" value="En" x="11.43" y="10.16" smashed="yes" rot="R180">
+<attribute name="VALUE" x="8.89" y="11.43" size="1.27" layer="27" rot="R270"/>
+</element>
 <element name="R4" library="resistor" package="R0805" value="82" x="11.43" y="15.24" rot="R90"/>
 <element name="Q1" library="basestation" package="SO8" value="SI4532ADY" x="25.4" y="19.05" rot="R270"/>
 <element name="R1" library="resistor" package="R0805" value="100K" x="16.51" y="19.05" rot="R270"/>
 <element name="R2" library="resistor" package="R0805" value="100K" x="27.94" y="24.765" rot="R90"/>
-<element name="F1" library="farnell-parts" package="1812" value="MF-MSMF110" x="36.83" y="30.48" rot="R270"/>
+<element name="F1" library="farnell-parts" package="1812" value="MF-MSMF110" x="36.83" y="25.4" smashed="yes" rot="R270">
+<attribute name="NAME" x="32.4758" y="26.0756" size="1.27" layer="25" rot="R270"/>
+</element>
 <element name="J2" library="farnell-parts" package="2-MOLEX" value="Bypass" x="31.75" y="5.08"/>
 <element name="J1" library="farnell-parts" package="2-MOLEX" value="En" x="25.4" y="5.08" smashed="yes">
@@
 <element name="J7" library="farnell-parts" package="2-MOLEX" value="LEN EN" x="19.05" y="5.08"/>
 <element name="J5" library="farnell-parts" package="2-MOLEX" value="12V Out" x="44.45" y="19.05" rot="R90"/>
-<element name="LED1" library="led" package="CHIP-LED0805" value="12V" x="6.35" y="10.16" rot="R180"/>
+<element name="LED1" library="led" package="CHIP-LED0805" value="12V" x="6.35" y="10.16" smashed="yes" rot="R180">
+<attribute name="VALUE" x="3.81" y="11.43" size="1.27" layer="27" rot="R270"/>
+</element>
 <element name="R3" library="resistor" package="R0805" value="680" x="6.35" y="15.24" rot="R90"/>
 <element name="C1" library="rcl" package="E5-13" value="2200uF" x="17.78" y="34.29" rot="R270"/>
@@
 </element>
 <element name="J4" library="farnell-parts" package="2-MOLEX" value="12v" x="5.08" y="21.59" rot="R270"/>
-<element name="J6" library="powerpoles" package="POWERPOLE_PAIR_25A" value="POWERPOLE_POWER25A" x="44.45" y="34.29" rot="R270"/>
+<element name="J6" library="powerpoles" package="POWERPOLE_PAIR_25A" value="POWERPOLE_POWER25A" x="44.45" y="34.29" rot="R90"/>
 <element name="J3" library="powerpoles" package="POWERPOLE_PAIR_25A" value="POWERPOLE_POWER25A" x="5.08" y="34.29" rot="R270"/>
 </elements>
@@
 <contactref element="J5" pad="2"/>
 <contactref element="J6" pad="RED"/>
-<wire x1="36.83" y1="31.905" x2="43.165" y2="38.24" width="1.6764" layer="1" curve="-90"/>
-<wire x1="43.165" y1="38.24" x2="43.6" y2="38.24" width="1.6764" layer="1"/>
-<wire x1="44.831" y1="20.32" x2="45.72" y2="20.32" width="1.6764" layer="1"/>
-<wire x1="45.72" y1="20.32" x2="48.26" y2="22.86" width="1.6764" layer="1" curve="90"/>
-<wire x1="48.26" y1="22.86" x2="48.26" y2="33.58" width="1.6764" layer="1"/>
-<wire x1="48.26" y1="33.58" x2="43.6" y2="38.24" width="1.6764" layer="1" curve="90"/>
+<wire x1="36.83" y1="26.825" x2="41.785" y2="26.825" width="1.6764" layer="1"/>
+<wire x1="41.785" y1="26.825" x2="45.3" y2="30.34" width="1.6764" layer="1" curve="90"/>
+<wire x1="41.785" y1="26.825" x2="44.831" y2="23.779" width="1.6764" layer="1" curve="-90"/>
+<wire x1="44.831" y1="23.779" x2="44.831" y2="20.32" width="1.6764" layer="1"/>
 </signal>
 <signal name="LEDGND">
@@
 <wire x1="17.78" y1="36.83" x2="20.32" y2="36.83" width="1.6764" layer="1"/>
 <wire x1="20.32" y1="36.83" x2="22.86" y2="34.29" width="1.6764" layer="1" curve="-90"/>
-<wire x1="22.86" y1="34.29" x2="22.86" y2="24.55" width="1.4224" layer="1"/>
+<wire x1="22.86" y1="34.29" x2="22.86" y2="24.55" width="1.6764" layer="1"/>
 <wire x1="6.35" y1="16.09" x2="6.35" y2="16.51" width="0.6096" layer="1"/>
 <wire x1="6.35" y1="16.51" x2="7.62" y2="17.78" width="0.6096" layer="1" curve="-90"/>
@@
 <wire x1="13.97" y1="38.78" x2="14.9" y2="39.71" width="0.6096" layer="1" curve="-90"/>
 <wire x1="22.86" y1="24.55" x2="23.71" y2="24.55" width="1.4224" layer="1"/>
-<wire x1="23.71" y1="24.55" x2="25.4" y2="22.86" width="1.4224" layer="1" curve="-90"/>
-<wire x1="25.4" y1="22.86" x2="25.4" y2="19.05" width="1.4224" layer="1"/>
+<wire x1="23.71" y1="24.55" x2="25.4" y2="22.86" width="1.6764" layer="1" curve="-90"/>
+<wire x1="25.4" y1="22.86" x2="25.4" y2="19.05" width="1.6764" layer="1"/>
 <wire x1="25.4" y1="19.05" x2="24.765" y2="18.415" width="1.4224" layer="1" curve="-90"/>
 <wire x1="24.765" y1="18.415" x2="22.8" y2="18.415" width="1.016" layer="1"/>
-<wire x1="30.48" y1="4.699" x2="30.48" y2="10.16" width="1.4224" layer="1"/>
-<wire x1="30.48" y1="10.16" x2="25.4" y2="15.24" width="1.4224" layer="1" curve="90"/>
-<wire x1="25.4" y1="15.24" x2="25.4" y2="19.05" width="1.4224" layer="1"/>
+<wire x1="30.48" y1="4.699" x2="30.48" y2="10.16" width="1.6764" layer="1"/>
+<wire x1="30.48" y1="10.16" x2="25.4" y2="15.24" width="1.6764" layer="1" curve="90"/>
+<wire x1="25.4" y1="15.24" x2="25.4" y2="19.05" width="1.6764" layer="1"/>
 <wire x1="27.94" y1="25.615" x2="24.775" y2="25.615" width="0.6096" layer="1"/>
 <wire x1="24.775" y1="25.615" x2="23.71" y2="24.55" width="0.6096" layer="1" curve="90"/>
@@
 <contactref element="Q1" pad="6"/>
 <contactref element="J2" pad="2"/>
-<wire x1="28" y1="17.145" x2="34.925" y2="17.145" width="1.4224" layer="1"/>
-<wire x1="34.925" y1="17.145" x2="36.83" y2="19.05" width="1.4224" layer="1" curve="90"/>
-<wire x1="36.83" y1="19.05" x2="36.83" y2="27.255" width="1.4224" layer="1"/>
-<wire x1="33.02" y1="4.699" x2="33.02" y2="15.24" width="1.4224" layer="1"/>
-<wire x1="33.02" y1="15.24" x2="34.925" y2="17.145" width="1.4224" layer="1" curve="-90"/>
+<wire x1="28" y1="17.145" x2="34.925" y2="17.145" width="1.6764" layer="1"/>
+<wire x1="34.925" y1="17.145" x2="36.83" y2="19.05" width="1.6764" layer="1" curve="90"/>
+<wire x1="33.02" y1="4.699" x2="33.02" y2="15.24" width="1.6764" layer="1"/>
+<wire x1="33.02" y1="15.24" x2="34.925" y2="17.145" width="1.6764" layer="1" curve="-90"/>
 <wire x1="28" y1="18.415" x2="28" y2="17.145" width="1.016" layer="1"/>
+<wire x1="36.83" y1="19.05" x2="36.83" y2="22.175" width="1.6764" layer="1"/>
 </signal>
 <signal name="N$2">
